File: pico-impa/pico-impa.kicad_pcb (KiCad board)
At the start: 2 copper layers, 94.5 x 94.7 mm, 32 parts, among them J1 Barrel_Jack_MountingPin, J2 Conn_01x10, J3 Conn_01x12, J4 Conn_01x10, U1 Raspberry Pi Pico, U2 Rasbperry Pi Pico Probe, U3 AMS1117-3.3, U4 LM35-LP, U5 ESP-01, U6 DHT11, U7 MPU9250, U8 SSD1306

Commit message: feat: pcb v1 finished
Routing:
- net VDC: track 40.0 -> 42.4 mm
- net (no net): vias 0 -> 3
- added copper zone on B.Cu, net GND
- added copper zone on F.Cu, net GND
Changed lines of the file:
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@@
     (style (thickness 0.05) (arrow_length 1.27) (text_position_mode 0) (extension_height 0.58642) (extension_offset 0.5) keep_text_aligned)
   )
+  (via (at 167.64 111.76) (size 5) (drill 5) (layers "F.Cu" "B.Cu") (free) (net 0))
+  (via (at 83.82 111.76) (size 5) (drill 5) (layers "F.Cu" "B.Cu") (free) (net 0))
+  (via (at 96.52 30.48) (size 5) (drill 5) (layers "F.Cu" "B.Cu") (free) (net 0))
   (segment (start 89.202527 87.63) (end 92.44 87.63) (width 1) (layer "B.Cu") (net 1))
   (segment (start 84.878489 83.305962) (end 89.202527 87.63) (width 1) (layer "B.Cu") (net 1))
@@
   (segment (start 92.805 90.17) (end 92.71 90.075) (width 1) (layer "B.Cu") (net 3))
   (segment (start 92.71 90.075) (end 87.551 90.075) (width 1) (layer "B.Cu") (net 3))
+  (segment (start 89.82 28.29) (end 91.567 26.543) (width 1) (layer "B.Cu") (net 4))
+  (segment (start 102.997 26.543) (end 104.38 27.926) (width 1) (layer "B.Cu") (net 4))
   (segment (start 119.38 29.845) (end 116.205 26.67) (width 1) (layer "B.Cu") (net 4))
+  (segment (start 91.567 26.543) (end 102.997 26.543) (width 1) (layer "B.Cu") (net 4))
   (segment (start 107.16 26.67) (end 104.38 29.45) (width 1) (layer "B.Cu") (net 4))
-  (segment (start 89.82 28.32) (end 103.25 28.32) (width 1) (layer "B.Cu") (net 4))
   (segment (start 121.92 29.845) (end 119.38 29.845) (width 1) (layer "B.Cu") (net 4))
   (segment (start 104.38 34.065) (end 104.605 34.29) (width 1) (layer "B.Cu") (net 4))
-  (segment (start 103.25 28.32) (end 104.38 29.45) (width 1) (layer "B.Cu") (net 4))
+  (segment (start 104.38 27.926) (end 104.38 29.45) (width 1) (layer "B.Cu") (net 4))
   (segment (start 104.38 31.09) (end 104.38 34.065) (width 1) (layer "B.Cu") (net 4))
   (segment (start 104.38 29.45) (end 104.38 31.09) (width 1) (layer "B.Cu") (net 4))
   (segment (start 116.205 26.67) (end 107.16 26.67) (width 1) (layer "B.Cu") (net 4))
+  (segment (start 89.82 28.32) (end 89.82 28.29) (width 1) (layer "B.Cu") (net 4))
   (segment (start 125.46 33.02) (end 126.365 33.02) (width 1) (layer "F.Cu") (net 5))
   (segment (start 126.365 33.02) (end 127 32.385) (width 1) (layer "F.Cu") (net 5))
@@
   (segment (start 121.79 57.899) (end 121.92 57.769) (width 1) (layer "F.Cu") (net 72))
   (segment (start 121.79 63.119) (end 121.79 57.899) (width 1) (layer "F.Cu") (net 72))
+  (zone (net 5) (net_name "GND") (layers F&B.Cu) (hatch edge 0.508)
+    (connect_pads (clearance 0.254))
+    (min_thickness 0.254) (filled_areas_thickness no)
+    (fill yes (thermal_gap 0.508) (thermal_bridge_width 0.508))
+    (polygon
+      (pts
+        (xy 173.101 116.713)
+        (xy 78.613 116.713)
+        (xy 78.613 21.971)
+        (xy 173.101 21.971)
+      )
+    )
+  )
 )
